Commit message: ajout cude dans l'environnement

File: src/hc10_moveit_config/urdf/hc10_macro.xacro (robot description, xacro)
@@ -174,4 +174,5 @@
       <axis xyz="0 0 1" />
       <limit lower="${radians(-180)}" upper="${radians(180)}" effort="368.48" velocity="${radians(130)}"/>
+      <dynamics damping="1.0" friction="1.0"/>
     </joint>
     <joint name="${prefix}joint_2_l" type="revolute">
@@ -181,4 +182,5 @@
       <axis xyz="0 1 0" />
       <limit lower="${radians(-180)}" upper="${radians(180)}" effort="368.48" velocity="${radians(130)}"/>
+      <dynamics damping="1.0" friction="1.0"/>
     </joint>
     <joint name="${prefix}joint_3_u" type="revolute">
@@ -188,4 +190,5 @@
       <axis xyz="0 -1 0" />
       <limit lower="${radians(-5)}" upper="${radians(355)}" effort="141.12" velocity="${radians(180)}"/>
+      <dynamics damping="1.0" friction="1.0"/>
     </joint>
     <joint name="${prefix}joint_4_r" type="revolute">
@@ -195,4 +198,5 @@
       <axis xyz="0 0 1" />
       <limit lower="${radians(-180)}" upper="${radians(180)}" effort="39.20" velocity="${radians(180)}"/>
+      <dynamics damping="1.0" friction="1.0"/>
     </joint>
     <joint name="${prefix}joint_5_b" type="revolute">
@@ -202,4 +206,5 @@
       <axis xyz="0 -1 0" />
       <limit lower="${radians(-180)}" upper="${radians(180)}" effort="31.36" velocity="${radians(250)}"/>
+      <dynamics damping="1.0" friction="1.0"/>
     </joint>
     <joint name="${prefix}joint_6_t" type="revolute">
@@ -209,4 +214,5 @@
       <axis xyz="0 0 1" />
       <limit lower="${radians(-180)}" upper="${radians(180)}" effort="31.36" velocity="${radians(250)}"/>
+      <dynamics damping="1.0" friction="1.0"/>
     </joint>
     <joint name="${prefix}joint_6_t-tool0" type="fixed">
