Commit message: Change cube size

File: src/hc10_moveit_config/urdf/hc10_cude_gazebo.xacro (robot description, xacro)
@@ -5,5 +5,5 @@
     <visual>
       <geometry>
-        <box size="0.2 0.2 0.2"/>
+        <box size="0.1 0.1 0.1"/>
       </geometry>
       <material name="Gazebo/Gray"/>
@@ -11,5 +11,5 @@
     <collision>
       <geometry>
-        <box size="0.2 0.2 0.2"/>
+        <box size="0.1 0.1 0.1"/>
       </geometry>
     </collision>
