Commit message: Start cleaning the code

File: src/hc10_moveit_config/urdf/hc10.xacro (robot description, xacro)
@@ -2,4 +2,6 @@
 <robot name="motoman_hc10" xmlns:xacro="http://ros.org/wiki/xacro">
   <xacro:include filename="$(find hc10_moveit_config)/urdf/hc10_macro.xacro" />
+  <xacro:include filename="$(find hc10_moveit_config)/urdf/hc10_gazebo.xacro" />
   <xacro:motoman_hc10 prefix=""/>
+  <xacro:gazebo_hc10 prefix=""/>
 </robot>

File: src/hc10_moveit_config/urdf/hc10_macro.xacro (robot description, xacro)
@@ -3,17 +3,4 @@
   <xacro:macro name="motoman_hc10" params="prefix">
     <xacro:include filename="$(find motoman_resources)/urdf/common_materials.xacro"/>
-    <xacro:macro name="control" params="joint">
-        <transmission name="${joint}_transmission">
-            <type>transmission_interface/SimpleTransmission</type>
-            <!-- The EffortJointInterface works best with Gazebo using torques to actuate the joints -->
-            <joint name="${joint}">
-                <hardwareInterface>hardware_interface/EffortJointInterface</hardwareInterface>
-            </joint>
-            <actuator name="${joint}_motor">
-                <hardwareInterface>hardware_interface/EffortJointInterface</hardwareInterface>
-                <mechanicalReduction>1</mechanicalReduction>
-            </actuator>
-        </transmission>
-    </xacro:macro>
     <!-- link list -->
     <link name="${prefix}base_link">
@@ -31,5 +18,5 @@
       <inertial>
         <origin xyz="0 0 0" rpy="0 0 0" />
-        <mass value="3.06" />
+        <mass value="0.1" />
         <inertia ixx="0.3" ixy="0.0" ixz="0.0" iyy="0.3" iyz="0.0" izz="0.3" />
       </inertial>
@@ -54,5 +41,5 @@
       <inertial>
         <origin xyz="0 0 0" rpy="0 0 0" />
-        <mass value="3.06" />
+        <mass value="0.1" />
         <inertia ixx="0.3" ixy="0.0" ixz="0.0" iyy="0.3" iyz="0.0" izz="0.3" />
       </inertial>
@@ -77,5 +64,5 @@
       <inertial>
         <origin xyz="0 0 0" rpy="0 0 0" />
-        <mass value="3.06" />
+        <mass value="0.1" />
         <inertia ixx="0.3" ixy="0.0" ixz="0.0" iyy="0.3" iyz="0.0" izz="0.3" />
       </inertial>
@@ -100,5 +87,5 @@
       <inertial>
         <origin xyz="0 0 0" rpy="0 0 0" />
-        <mass value="3.06" />
+        <mass value="0.1" />
         <inertia ixx="0.3" ixy="0.0" ixz="0.0" iyy="0.3" iyz="0.0" izz="0.3" />
       </inertial>
@@ -123,5 +110,5 @@
       <inertial>
         <origin xyz="0 0 0" rpy="0 0 0" />
-        <mass value="3.06" />
+        <mass value="0.1" />
         <inertia ixx="0.3" ixy="0.0" ixz="0.0" iyy="0.3" iyz="0.0" izz="0.3" />
       </inertial>
@@ -146,5 +133,5 @@
       <inertial>
         <origin xyz="0 0 0" rpy="0 0 0" />
-        <mass value="3.06" />
+        <mass value="0.1" />
         <inertia ixx="0.3" ixy="0.0" ixz="0.0" iyy="0.3" iyz="0.0" izz="0.3" />
       </inertial>
@@ -169,5 +156,5 @@
       <inertial>
         <origin xyz="0 0 0" rpy="0 0 0" />
-        <mass value="3.06" />
+        <mass value="0.1" />
         <inertia ixx="0.3" ixy="0.0" ixz="0.0" iyy="0.3" iyz="0.0" izz="0.3" />
       </inertial>
@@ -187,7 +174,5 @@
       <axis xyz="0 0 1" />
       <limit lower="${radians(-180)}" upper="${radians(180)}" effort="368.48" velocity="${radians(130)}"/>
-      <dynamics damping="1.0" friction="1.0"/>
-    </joint>
-    <xacro:control joint="${prefix}joint_1_s"/>
+    </joint>
     <joint name="${prefix}joint_2_l" type="revolute">
       <parent link="${prefix}link_1_s"/>
@@ -196,7 +181,5 @@
       <axis xyz="0 1 0" />
       <limit lower="${radians(-180)}" upper="${radians(180)}" effort="368.48" velocity="${radians(130)}"/>
-      <dynamics damping="1.0" friction="1.0"/>
-    </joint>
-    <xacro:control joint="${prefix}joint_2_l"/>
+    </joint>
     <joint name="${prefix}joint_3_u" type="revolute">
       <parent link="${prefix}link_2_l"/>
@@ -205,7 +188,5 @@
       <axis xyz="0 -1 0" />
       <limit lower="${radians(-5)}" upper="${radians(355)}" effort="141.12" velocity="${radians(180)}"/>
-      <dynamics damping="1.0" friction="1.0"/>
-    </joint>
-    <xacro:control joint="${prefix}joint_3_u"/>
+    </joint>
     <joint name="${prefix}joint_4_r" type="revolute">
       <parent link="${prefix}link_3_u"/>
@@ -214,7 +195,5 @@
       <axis xyz="0 0 1" />
       <limit lower="${radians(-180)}" upper="${radians(180)}" effort="39.20" velocity="${radians(180)}"/>
-      <dynamics damping="1.0" friction="1.0"/>
-    </joint>
-    <xacro:control joint="${prefix}joint_4_r"/>
+    </joint>
     <joint name="${prefix}joint_5_b" type="revolute">
       <parent link="${prefix}link_4_r"/>
@@ -223,7 +202,5 @@
       <axis xyz="0 -1 0" />
       <limit lower="${radians(-180)}" upper="${radians(180)}" effort="31.36" velocity="${radians(250)}"/>
-      <dynamics damping="1.0" friction="1.0"/>
-    </joint>
-    <xacro:control joint="${prefix}joint_5_b"/>
+    </joint>
     <joint name="${prefix}joint_6_t" type="revolute">
       <parent link="${prefix}link_5_b"/>
@@ -232,7 +209,5 @@
       <axis xyz="0 0 1" />
       <limit lower="${radians(-180)}" upper="${radians(180)}" effort="31.36" velocity="${radians(250)}"/>
-      <dynamics damping="1.0" friction="1.0"/>
-    </joint>
-    <xacro:control joint="${prefix}joint_6_t"/>
+    </joint>
     <joint name="${prefix}joint_6_t-tool0" type="fixed">
       <origin xyz="0 0 -0.130" rpy="${pi} 0 0"/>
@@ -249,13 +224,4 @@
       <child link="${prefix}base"/>
     </joint>
-    <link name="world"/>
-    <joint name="world_joint" type="fixed">
-      <origin xyz="0 0 0" rpy="0 0 0"/>  <!-- Place the robot wherever you want -->
-      <parent link="world"/>
-      <child link="${prefix}base_link"/>  <!-- replace this name with your robot's base link -->
-    </joint>
   </xacro:macro>
-  <gazebo>
-      <plugin name="gazebo_ros_control" filename="libgazebo_ros_control.so"/>
-  </gazebo>
 </robot>

Commit message: Ajout capteur

File: src/hc10_moveit_config/urdf/hc10.xacro (robot description, xacro)
@@ -3,3 +3,21 @@
   <xacro:include filename="$(find hc10_moveit_config)/urdf/hc10_macro.xacro" />
   <xacro:motoman_hc10 prefix=""/>
+  <xacro:include filename="$(find hc10_moveit_config)/urdf/kinect.urdf.xacro" />
+  <xacro:sensor_hc10 prefix=""/>
+  <link name="camera_depth_frame">
+    <visual>
+      <geometry>
+        <box size="0.05 0.2 0.05"/>
+      </geometry>
+      <material name="Kinect_gray">
+        <color rgba="0.2 0.2 0.2 1.0"/>
+      </material>
+    </visual>
+  </link>
+  <!-- Attach Kinect to base -->
+  <joint name="tool0-camera" type="fixed">
+    <origin xyz="0 0 -0.130" rpy="${pi} 0 0"/>
+    <parent link="tool0"/>
+    <child link="camera_depth_frame"/>
+  </joint>
 </robot>

Commit message: positionnement de la kinect sur l'organe terminal

File: src/hc10_moveit_config/urdf/hc10.xacro (robot description, xacro)
@@ -8,5 +8,5 @@
     <visual>
       <geometry>
-        <box size="0.05 0.2 0.05"/>
+        <box size="0.2 0.05 0.02"/>
       </geometry>
       <material name="Kinect_gray">
@@ -17,5 +17,5 @@
   <!-- Attach Kinect to base -->
   <joint name="tool0-camera" type="fixed">
-    <origin xyz="0 0 -0.130" rpy="${pi} 0 0"/>
+    <origin xyz="0 0 0.01" rpy="${pi} 0 0"/>
     <parent link="tool0"/>
     <child link="camera_depth_frame"/>

Commit message: modif du nom de parent link

File: src/hc10_moveit_config/urdf/hc10.xacro (robot description, xacro)
@@ -17,5 +17,5 @@
   <!-- Attach Kinect to base -->
   <joint name="tool0-camera" type="fixed">
-    <origin xyz="0 0 0.01" rpy="${pi} 0 0"/>
+    <origin xyz="0 0 0.01" rpy="${pi} ${-pi/2} 0"/>
     <parent link="tool0"/>
     <child link="camera_depth_frame"/>

Commit message: Affichage nuage de point dans Rviz

File: src/hc10_moveit_config/urdf/hc10.xacro (robot description, xacro)
@@ -10,5 +10,5 @@
     <visual>
       <geometry>
-        <box size="0.2 0.05 0.02"/>
+        <box size="0.03 0.02 0.08"/>
       </geometry>
       <material name="Kinect_gray">
@@ -19,5 +19,5 @@
   <!-- Attach Kinect to base -->
   <joint name="tool0-camera" type="fixed">
-    <origin xyz="0 0 0.01" rpy="${pi} ${-pi/2} 0"/>
+    <origin xyz="0.0 -0.0 0.015" rpy="${pi} ${-pi/2} 0"/>
     <parent link="tool0"/>
     <child link="camera_depth_frame"/>
